Commit message: tom - updating from nuc

File: my_robot/urdf/make_block_r.urdf (robot description, URDF)
Before this commit: robot My_Robot, 6 links, 5 joints
Links:
- added link fcu; visual box size=.085 .052 .02
Joints:
- added joint base_to_fcu: type fixed, parent base_link, child fcu, origin xyz=0 0 0.26 rpy=0 0 0
